File: MB.kicad_sch (KiCad schematic)
At the start: 4 parts

Commit message: routing pcb complete
Parts:
- gave numbers to parts that had none: 4
Other:
- added sheet RELAYS_2 (RELAYS_2.kicad_sch)
- note added: "[3] RELAYS 1"
- note added: "[4] RELAYS 2"
- note removed: "[3] RELAYS"
- moved on the sheet: H1, H2, H3, H4
