File: MCU.kicad_sch (KiCad schematic)
At the start: 14 parts, among them J200 Serial Wire Debug, U200 STM32F103C8Tx, Y200 16MHz

Commit message: routing pcb complete
Parts:
- removed TP?: TestPoint, TestPoint:TestPoint_Pad_D2.0mm, symbol Connector:TestPoint
- added H100: WIZ850IO, WIZ850:WIZ850IO, symbol WIZ850IO:WIZ850IO
Connections:
- net +3V3: now also H100.8 (3.3V_1), H100.9 (3.3V_2)
- net GND: now also H100.1 (GND_1), H100.2 (GND_2), H100.7 (GND_3)
- net SCLK: now also U200.37 (PA14)
- net SWDIO: now also U200.34 (PA13)
- net ETH_RST: now reaches U200.13 (PA3)
- net ETH_RST: now also H100.11 (RSTN)
- net ETH_SCK: now reaches U200.15 (PA5)
- net ETH_SCK: now also H100.4 (SCLK)
- net ETH_MISO: now reaches U200.16 (PA6)
- net ETH_MISO: now also H100.12 (MISO)
- net ETH_MOSI: now reaches U200.17 (PA7)
- net ETH_MOSI: now also H100.3 (MOSI)
- net ETH_CS: now reaches U200.18 (PB0)
- net ETH_CS: now also H100.5 (SCNN)
- net 9_TECHO: now reaches U200.19 (PB1)
- net 9_MESA: now reaches U200.20 (PB2)
- net 8_TECHO: now reaches U200.25 (PB12)
- net 8_MESA: now reaches U200.26 (PB13)
- net 7_TECHO: now reaches U200.27 (PB14)
- net 7_MESA: now reaches U200.28 (PB15)
- net 6_TECHO: now reaches U200.29 (PA8)
- net 6_MESA: now reaches U200.30 (PA9)
- net 5_TECHO: now reaches U200.31 (PA10)
- net 1_MESA: now reaches U200.32 (PA11)
- net 1_TECHO: now reaches U200.38 (PA15)
- net 2_MESA: now reaches U200.39 (PB3)
- net 2_TECHO: now reaches U200.40 (PB4)
- net 3_MESA: now reaches U200.41 (PB5)
- net 3_TECHO: now reaches U200.42 (PB6)
- net 4_MESA: now reaches U200.43 (PB7)
- net 4_TECHO: now reaches U200.45 (PB8)
- net 5_MESA: now reaches U200.46 (PB9)
- no-connect marks 0 -> 1
Other:
- note added: "ETHERNET MODULE WIZ850"
- moved on the sheet: C200, C201, C202, C203, C204, C205, C206, C207, J200, R200, S200, U200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
