File: RELAYS.kicad_sch (KiCad schematic)
At the start: 9 parts

Commit message: routing pcb complete
Parts:
- removed D?: SMF24A-TP, Jose_:SOD_123FL, symbol Device:D_Schottky
- added D304, D307, D310, D313, D316, D319, D322, D325, D328: SM4007PL, Jose_:SOD_123FL, symbol Device:D_Zener
- added D305, D308, D311, D314, D317, D320, D323, D326, D329: LED_DOOR, LED_SMD:LED_0603_1608Metric, symbol Device:LED
- added J301, J303, J305, J307, J309: TECHO_OUTPUT, Connector_Phoenix_MSTB:PhoenixContact_MSTBA_2,5_2-G-5,08_1x02_P5.08mm_Horizontal, symbol Connector:Screw_Terminal_01x02
- added J302, J304, J306, J308: MESA_OUTPUT, Connector_Phoenix_MSTB:PhoenixContact_MSTBA_2,5_2-G-5,08_1x02_P5.08mm_Horizontal, symbol Connector:Screw_Terminal_01x02
- added K301, K302, K303, K304, K305, K306, K307, K308, K309: HF49FD/005-1H12T, HF49FD_005-1H11F:HF49FD0051H11F, symbol HF49FD_005-1H12T:HF49FD/005-1H12T
- added Q301, Q302, Q303, Q304, Q305, Q306, Q307, Q308, Q309: MMBT3904, Package_TO_SOT_SMD:SOT-23, symbol Transistor_BJT:MMBT5550L
- added R303, R306, R309, R312, R315, R318, R321, R324, R327: 1k, Resistor_SMD:R_0603_1608Metric, symbol Device:R_Small
- added R304, R307, R310, R313, R316, R319, R322, R325, R328: 1K, Resistor_SMD:R_0603_1608Metric, symbol Device:R_Small
- added R305, R308, R311, R314, R317, R320, R323, R326, R329: 10K, Resistor_SMD:R_0603_1608Metric, symbol Device:R_Small
- J300: renamed from J?; value DOOR_OUTPUT -> MESA_OUTPUT
- K300: renamed from K?; footprint HF49_RELAY:RELAY_HF49FD_005-1H12T -> HF49FD_005-1H11F:HF49FD0051H11F
- gave numbers to parts that had none: 6
Connections:
- net +5V: now also D304.1 (K), D307.1 (K), D310.1 (K), D313.1 (K), D316.1 (K), D319.1 (K), D322.1 (K), D325.1 (K), D328.1 (K), K301.2, K302.2, K303.2, K304.2, K305.2, K306.2, K307.2, K308.2, K309.2, R303.2, R306.2, R309.2, R312.2, R315.2, R318.2, R321.2, R324.2, R327.2
- net GND: now also Q301.2 (E), Q302.2 (E), Q303.2 (E), Q304.2 (E), Q305.2 (E), Q306.2 (E), Q307.2 (E), Q308.2 (E), Q309.2 (E), R305.1, R308.1, R311.1, R314.1, R317.1, R320.1, R323.1, R326.1, R329.1; no longer J300.1 (Pin_1)
- net +24V: no longer names the net of K300.4
- net +24V: now also J300.1 (Pin_1)
- net COIL_1: no longer names the net of D301.2 (A), D302.1 (K), K300.1, Q300.3 (C)
- net DOOR_PIN renamed 1_MESA
- net RELAY_24V: no longer names the net of J300.2 (Pin_2), K300.3
- new net: Q304.1 (B), R313.2
- new net: D313.2 (A), D314.1 (K), K304.1, Q304.3 (C)
- new net: D305.2 (A), R303.1
- new net: Q302.1 (B), R307.2
- new net: D323.2 (A), R321.1
- new net: J303.1 (Pin_1), K303.4
- new net: J303.2 (Pin_2), K303.3
- new net: Q301.1 (B), R304.2
- new net: D304.2 (A), D305.1 (K), K301.1, Q301.3 (C)
- new net: D316.2 (A), D317.1 (K), K305.1, Q305.3 (C)
- new net: D317.2 (A), R315.1
- new net: J305.2 (Pin_2), K305.3
- new net: J305.1 (Pin_1), K305.4
- new net: Q303.1 (B), R310.2
- new net: Q308.1 (B), R325.2
- new net: D325.2 (A), D326.1 (K), K308.1, Q308.3 (C)
- new net: D322.2 (A), D323.1 (K), K307.1, Q307.3 (C)
- new net: D326.2 (A), R324.1
- new net: D319.2 (A), D320.1 (K), K306.1, Q306.3 (C)
- new net: J301.2 (Pin_2), K301.3
- new net: J301.1 (Pin_1), K301.4
- new net: D310.2 (A), D311.1 (K), K303.1, Q303.3 (C)
- new net: D308.2 (A), R306.1
- new net: D320.2 (A), R318.1
- new net: J307.2 (Pin_2), K307.3
- new net: J307.1 (Pin_1), K307.4
- new net: J302.1 (Pin_1), K302.4
- new net: J302.2 (Pin_2), K302.3
- new net: J309.1 (Pin_1), K309.4
- new net: J309.2 (Pin_2), K309.3
- new net: D328.2 (A), D329.1 (K), K309.1, Q309.3 (C)
- new net: D329.2 (A), R327.1
- new net: D314.2 (A), R312.1
- new net: Q305.1 (B), R316.2
- new net: J308.1 (Pin_1), K308.4
- new net: J308.2 (Pin_2), K308.3
- new net: Q307.1 (B), R322.2
- new net: Q309.1 (B), R328.2
- new net: J306.2 (Pin_2), K306.3
- new net: J306.1 (Pin_1), K306.4
- new net: D307.2 (A), D308.1 (K), K302.1, Q302.3 (C)
- new net: Q306.1 (B), R319.2
- new net: J304.2 (Pin_2), K304.3
- new net: J304.1 (Pin_1), K304.4
- new net: D311.2 (A), R309.1
- new net 1_TECHO: R304.1, R305.2
- new net 2_MESA: R307.1, R308.2
- new net 2_TECHO: R310.1, R311.2
- new net 3_MESA: R313.1, R314.2
- new net 3_TECHO: R316.1, R317.2
- new net 4_MESA: R319.1, R320.2
- new net 4_TECHO: R322.1, R323.2
- new net 5_MESA: R325.1, R326.2
- new net 5_TECHO: R328.1, R329.2
Other:
- note added: "CABINA 1 / CABINA 10 LUCES MESA Y TECHO"
- note added: "CABINA 2 / CABINA 11 LUCES MESA Y TECHO"
- note added: "CABINA 3 / CABINA 12 LUCES MESA Y TECHO"
- note added: "CABINA 4 / CABINA 13 LUCES MESA Y TECHO"
- note added: "CABINA 5 / CABINA 14 LUCES MESA Y TECHO"
- note removed: "RELAY DRIVER FOR DOOR"
- moved on the sheet: D301, D302, J300, K300, Q300, R300, R301, R302
