File: POWER.kicad_sch (KiCad schematic)
At the start: 27 parts, among them J100 VCC INPUT, J101 SWITCH ON/OFF, J102 FAN VOLTAGE, Q100 WST4045, U100 LMR23625CFDDA, U101 AMS1117-3.3

Commit message: routing pcb complete
Parts:
- added C106: 22u, Capacitor_SMD:C_0805_2012Metric, symbol Device:C
- C100: footprint (none) -> Capacitor_SMD:C_Elec_6.3x7.7; LCSC (none) -> C445060
- C101: footprint (none) -> Capacitor_SMD:C_1210_3225Metric; LCSC (none) -> C694199
- C102: footprint (none) -> Capacitor_SMD:C_0603_1608Metric; LCSC (none) -> C342915
- C103: value 10p -> 2.2u; footprint (none) -> Capacitor_SMD:C_0603_1608Metric; LCSC (none) -> C385892
- C104: footprint (none) -> Capacitor_SMD:C_0805_2012Metric; LCSC (none) -> C1854115
- C105: value 47u -> 22u; footprint (none) -> Capacitor_SMD:C_0805_2012Metric; LCSC (none) -> C380338
- L100: footprint (none) -> Jose_:SMD_I_6.6x7.1mm; LCSC (none) -> C2847482
- R101: footprint (none) -> Resistor_SMD:R_0603_1608Metric; LCSC (none) -> C728599
- R102: footprint (none) -> Resistor_SMD:R_0603_1608Metric; LCSC (none) -> C137768
- U100: footprint LMR23625CFDDA:VREG_LM5017MR/NOPB -> LMR23625:VREG_LM5017MR_NOPB
- renumbered C106 to C107, C107 to C108
Connections:
- net +24V: now also C100.1, C101.1, U100.5 (EN/SYNC), U100.7 (VIN)
- net +5V: now also C106.1
- net GND: now also J100.2 (Pin_2), U100.9 (GND_PAD), C106.2; no longer J100.1 (Pin_1)
- net V_INPUT: now also J100.1 (Pin_1); no longer J100.2 (Pin_2)
Other:
- moved on the sheet: D102, J100

Commit message: change switch position and thermal vias of LMR
Parts:
- U100: Availability In Stock -> (none); Check_prices https://www.snapeda.com/parts/LMR23625CFDDA/Texas+Instrumen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 -> (none); LCSC (none) -> C2070635; MF Texas Instruments -> (none); MP LMR23625CFDDA -> (none); Package HSOIC-8 Texas Instruments -> (none); Price None -> (none); Purchase-URL https://www.snapeda.com/api/url_track_click_mouser/?unipart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 -> (none); SnapEDA_Link https://www.snapeda.com/parts/LMR23625CFDDA/Texas+Instrumen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 -> (none)
Changed lines of the file:
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@@
       (effects (font (size 1.27 1.27)) hide)
     )
-    (property "MF" "Texas Instruments" (id 4) (at 157.988 73.914 0)
-      (effects (font (size 1.27 1.27)) (justify bottom) hide)
-    )
-    (property "Description" "\nSIMPLE SWITCHER®, 36V 2.5A Synchronous Step-Down Converter\n" (id 5) (at 157.988 73.914 0)
-      (effects (font (size 1.27 1.27)) (justify bottom) hide)
-    )
-    (property "Package" "HSOIC-8 Texas Instruments" (id 6) (at 157.988 73.914 0)
-      (effects (font (size 1.27 1.27)) (justify bottom) hide)
-    )
-    (property "Price" "None" (id 7) (at 157.988 73.914 0)
-      (effects (font (size 1.27 1.27)) (justify bottom) hide)
-    )
-    (property "SnapEDA_Link" "https://www.snapeda.com/parts/LMR23625CFDDA/Texas+Instruments/view-part/?ref=snap" (id 8) (at 157.988 73.914 0)
-      (effects (font (size 1.27 1.27)) (justify bottom) hide)
-    )
-    (property "MP" "LMR23625CFDDA" (id 9) (at 157.988 73.914 0)
-      (effects (font (size 1.27 1.27)) (justify bottom) hide)
-    )
-    (property "Purchase-URL" "https://www.snapeda.com/api/url_track_click_mouser/?unipart_id=1241541&manufacturer=Texas Instruments&part_name=LMR23625CFDDA&search_term=lmr23625" (id 10) (at 157.988 73.914 0)
-      (effects (font (size 1.27 1.27)) (justify bottom) hide)
-    )
-    (property "Availability" "In Stock" (id 11) (at 157.988 73.914 0)
-      (effects (font (size 1.27 1.27)) (justify bottom) hide)
-    )
-    (property "Check_prices" "https://www.snapeda.com/parts/LMR23625CFDDA/Texas+Instruments/view-part/?ref=eda" (id 12) (at 157.988 73.914 0)
-      (effects (font (size 1.27 1.27)) (justify bottom) hide)
+    (property "LCSC" "C2070635" (id 4) (at 157.988 73.914 0)
+      (effects (font (size 1.27 1.27)) hide)
     )
     (pin "1")
